File: Electrical/KiCad_templates/Expansion_Card_Retrofit/Expansion_Card_Retrofit.kicad_pcb (KiCad board)
At the start: 4 copper layers, 26 x 30 mm, 49 parts, among them J1 Conn 10P, P1 USB_C_Plug_USB2.0, Q1 DMG1012T, Q2 Q_PMOS_SGD, Q3 Q_Dual_NPN_NPN_C2E2C1E1B1B2, U1 AP7366EA-3.3, U2 RP2040, U3 W25Q16JVUXIQ, U4 RP2040, U5 W25Q16JVUXIQ, X1 ECS-2520MVLC-120-CM-TR

Commit message: Added test points
Parts:
- added R2: 1K, Resistor_SMD:R_0402_1005Metric, F.Cu at (135.3, 106.9)
- added TP5: BOOT, TestPoint:TestPoint_Pad_1.0x1.0mm, B.Cu at (133.6, 107.4)
- added TP7: RST2, TestPoint:TestPoint_Pad_1.0x1.0mm, B.Cu at (139.2, 93.5)
- added TP8: RST1, TestPoint:TestPoint_Pad_1.0x1.0mm, B.Cu at (148.4, 99.7)
Connections:
- U4 pad 26: unconnected-(U4-RUN-Pad26) -> Net-(U4-RUN)
Routing:
- net Net-(U4-RUN): track 0.00 -> 2.70 mm, vias 0 -> 1
- net Net-(R2-Pad1): track 0.00 -> 1.70 mm, vias 0 -> 1
- net /Development Board Section/RUN: track 17.7 -> 19.4 mm
- net +3V3: track 63.7 -> 64.4 mm, vias 15 -> 16
- net USB_D_P: track 9.42 -> 8.73 mm
- net USB_D_N: track 9.59 -> 9.00 mm
- net GND: vias 68 -> 66

Commit message: Production design v1 finished
Parts:
- added C1: 10u, Capacitor_SMD:C_0402_1005Metric, F.Cu at (154.3, 132.3)
- added C1: 10u, Capacitor_SMD:C_0402_1005Metric, F.Cu at (126.3, 132.3)
- added C1: 10u, Capacitor_SMD:C_0402_1005Metric, F.Cu at (143.7, 78.7)
- added C10: 100n, Capacitor_SMD:C_0201_0603Metric, F.Cu at (140.5, 91.7)
- added C10: 100n, Capacitor_SMD:C_0201_0603Metric, F.Cu at (129.5, 119.3)
- added C10: 100n, Capacitor_SMD:C_0201_0603Metric, F.Cu at (157.5, 119.3)
- added C11: 100n, Capacitor_SMD:C_0201_0603Metric, F.Cu at (132.3, 125.2)
- added C11: 100n, Capacitor_SMD:C_0201_0603Metric, F.Cu at (160.3, 125.2)
- added C11: 100n, Capacitor_SMD:C_0201_0603Metric, F.Cu at (137.7, 85.8)
- added C12: 100n, Capacitor_SMD:C_0201_0603Metric, F.Cu at (142.0, 119.0)
- added C12: 100n, Capacitor_SMD:C_0201_0603Metric, F.Cu at (114.0, 119.0)
- added C12: 100n, Capacitor_SMD:C_0201_0603Metric, F.Cu at (156.0, 92.0)
- added C13: 100n, Capacitor_SMD:C_0201_0603Metric, F.Cu at (144.7, 130.2)
- added C13: 100n, Capacitor_SMD:C_0201_0603Metric, F.Cu at (116.7, 130.2)
- added C13: 100n, Capacitor_SMD:C_0201_0603Metric, F.Cu at (153.3, 80.8)
- added C14: 2u2, Capacitor_SMD:C_0402_1005Metric, F.Cu at (112.3, 129.8)
- added C14: 2u2, Capacitor_SMD:C_0402_1005Metric, F.Cu at (140.3, 129.8)
- added C14: 2u2, Capacitor_SMD:C_0402_1005Metric, F.Cu at (157.7, 81.2)
- added C15: 2u2, Capacitor_SMD:C_0402_1005Metric, F.Cu at (138.8, 129.8)
- added C15: 2u2, Capacitor_SMD:C_0402_1005Metric, F.Cu at (110.8, 129.8)
- added C15: 2u2, Capacitor_SMD:C_0402_1005Metric, F.Cu at (159.2, 81.2)
- added C16: 100n, Capacitor_SMD:C_0201_0603Metric, F.Cu at (149.0, 83.8)
- added C16: 100n, Capacitor_SMD:C_0201_0603Metric, F.Cu at (121.0, 127.2)
- added C16: 100n, Capacitor_SMD:C_0201_0603Metric, F.Cu at (149.0, 127.2)
- added C18: 1n, Capacitor_SMD:C_0201_0603Metric, F.Cu at (119.1, 118.3)
- added C18: 1n, Capacitor_SMD:C_0201_0603Metric, F.Cu at (150.9, 92.7)
- added C18: 1n, Capacitor_SMD:C_0201_0603Metric, F.Cu at (147.1, 118.3)
- added C19: 100n, Capacitor_SMD:C_0201_0603Metric, F.Cu at (149.0, 123.2)
- added C19: 100n, Capacitor_SMD:C_0201_0603Metric, F.Cu at (149.0, 87.8)
- added C19: 100n, Capacitor_SMD:C_0201_0603Metric, F.Cu at (121.0, 123.2)
- added C2: 10u, Capacitor_SMD:C_0402_1005Metric, F.Cu at (130.4, 134.8)
- added C2: 10u, Capacitor_SMD:C_0402_1005Metric, F.Cu at (139.6, 76.2)
- added C2: 10u, Capacitor_SMD:C_0402_1005Metric, F.Cu at (158.4, 134.8)
- added C20: 100n, Capacitor_SMD:C_0201_0603Metric, F.Cu at (154.8, 92.0)
- added C20: 100n, Capacitor_SMD:C_0201_0603Metric, F.Cu at (115.2, 119.0)
- added C20: 100n, Capacitor_SMD:C_0201_0603Metric, F.Cu at (143.2, 119.0)
- added C21: 100n, Capacitor_SMD:C_0201_0603Metric, F.Cu at (111.0, 123.7)
- added C21: 100n, Capacitor_SMD:C_0201_0603Metric, F.Cu at (139.0, 123.7)
- added C21: 100n, Capacitor_SMD:C_0201_0603Metric, F.Cu at (159.0, 87.3)
- added C22: 100n, Capacitor_SMD:C_0201_0603Metric, F.Cu at (146.2, 91.5)
- added C22: 100n, Capacitor_SMD:C_0201_0603Metric, F.Cu at (151.8, 119.5)
- added C22: 100n, Capacitor_SMD:C_0201_0603Metric, F.Cu at (123.8, 119.5)
- added C24: 100n, Capacitor_SMD:C_0201_0603Metric, F.Cu at (124.7, 129.3)
- added C24: 100n, Capacitor_SMD:C_0201_0603Metric, F.Cu at (152.7, 129.3)
- added C24: 100n, Capacitor_SMD:C_0201_0603Metric, F.Cu at (145.3, 81.7)
- added C5: 100n, Capacitor_SMD:C_0201_0603Metric, F.Cu at (149.0, 86.2)
- added C5: 100n, Capacitor_SMD:C_0201_0603Metric, F.Cu at (121.0, 124.8)
- added C5: 100n, Capacitor_SMD:C_0201_0603Metric, F.Cu at (149.0, 124.8)
- added C6: 100n, Capacitor_SMD:C_0201_0603Metric, F.Cu at (131.0, 125.2)
- added C6: 100n, Capacitor_SMD:C_0201_0603Metric, F.Cu at (159.0, 125.2)
- added C6: 100n, Capacitor_SMD:C_0201_0603Metric, F.Cu at (139.0, 85.8)
- added C7: 2u2, Capacitor_SMD:C_0402_1005Metric, F.Cu at (132.6, 127.3)
- added C7: 2u2, Capacitor_SMD:C_0402_1005Metric, F.Cu at (160.6, 127.3)
- added C7: 2u2, Capacitor_SMD:C_0402_1005Metric, F.Cu at (137.4, 83.7)
- added C8: 2u2, Capacitor_SMD:C_0402_1005Metric, F.Cu at (159.1, 127.3)
- added C8: 2u2, Capacitor_SMD:C_0402_1005Metric, F.Cu at (138.9, 83.7)
- added C8: 2u2, Capacitor_SMD:C_0402_1005Metric, F.Cu at (131.1, 127.3)
- added C9: 2u2, Capacitor_SMD:C_0402_1005Metric, F.Cu at (132.6, 129.7)
- added C9: 2u2, Capacitor_SMD:C_0402_1005Metric, F.Cu at (137.4, 81.3)
- added C9: 2u2, Capacitor_SMD:C_0402_1005Metric, F.Cu at (160.6, 129.7)
- added D1: Green, LED_SMD:LED_0402_1005Metric, F.Cu at (110.0, 106.8)
- added D1: Green, LED_SMD:LED_0402_1005Metric, F.Cu at (138.0, 106.8)
- added D1: Green, LED_SMD:LED_0402_1005Metric, F.Cu at (160.0, 104.2)
- added D2: Orange, LED_SMD:LED_0402_1005Metric, F.Cu at (115.2, 132.8)
- added D2: Orange, LED_SMD:LED_0402_1005Metric, F.Cu at (143.2, 132.8)
- added D2: Orange, LED_SMD:LED_0402_1005Metric, F.Cu at (154.8, 78.2)
- added H1: MountingHole, MountingHole:MountingHole_2.2mm_M2, F.Cu at (160.3, 116.5)
- added H1: MountingHole, MountingHole:MountingHole_2.2mm_M2, F.Cu at (132.3, 116.5)
- added H1: MountingHole, MountingHole:MountingHole_2.2mm_M2, F.Cu at (137.7, 94.5)
- added H2: MountingHole, MountingHole:MountingHole_2.2mm_M2, F.Cu at (137.7, 116.5)
- added H2: MountingHole, MountingHole:MountingHole_2.2mm_M2, F.Cu at (160.3, 94.5)
- added H2: MountingHole, MountingHole:MountingHole_2.2mm_M2, F.Cu at (109.7, 116.5)
- added J1: Conn 10P, SnapEDA:Pinheader_PCB_Edge_2x5_2.54mm, F.Cu at (151.9, 101.2)
- added J1: Conn 10P, SnapEDA:Pinheader_PCB_Edge_2x5_2.54mm, F.Cu at (146.1, 109.8)
- added J1: Conn 10P, SnapEDA:Pinheader_PCB_Edge_2x5_2.54mm, F.Cu at (118.1, 109.8)
- added P1: USB_C_Plug_USB2.0, Expansion_Card:USB_C_Plug_Molex_105444, F.Cu at (149.0, 77.0)
- added P1: USB_C_Plug_USB2.0, Expansion_Card:USB_C_Plug_Molex_105444, F.Cu at (149.0, 134.0)
- added P1: USB_C_Plug_USB2.0, Expansion_Card:USB_C_Plug_Molex_105444, F.Cu at (121.0, 134.0)
- added Q1: DMG1012T, Package_DFN_QFN:Diodes_DFN1006-3, F.Cu at (148.4, 92.0)
- added Q1: DMG1012T, Package_DFN_QFN:Diodes_DFN1006-3, F.Cu at (149.6, 119.0)
- added Q1: DMG1012T, Package_DFN_QFN:Diodes_DFN1006-3, F.Cu at (121.6, 119.0)
- added Q2: Q_PMOS_SGD, Package_TO_SOT_SMD:SOT-723, F.Cu at (141.5, 96.5)
- added Q2: Q_PMOS_SGD, Package_TO_SOT_SMD:SOT-723, F.Cu at (156.5, 114.5)
- added Q2: Q_PMOS_SGD, Package_TO_SOT_SMD:SOT-723, F.Cu at (128.5, 114.5)
- added Q3: Q_Dual_NPN_NPN_C2E2C1E1B1B2, digikey-footprints:SOT-363, F.Cu at (154.6, 117.3)
- added Q3: Q_Dual_NPN_NPN_C2E2C1E1B1B2, digikey-footprints:SOT-363, F.Cu at (126.6, 117.3)
- added Q3: Q_Dual_NPN_NPN_C2E2C1E1B1B2, digikey-footprints:SOT-363, F.Cu at (143.4, 93.7)
- added R1: 5k1, Resistor_SMD:R_0402_1005Metric, F.Cu at (147.5, 80.5)
- added R1: 5k1, Resistor_SMD:R_0402_1005Metric, F.Cu at (150.5, 130.6)
- added R1: 5k1, Resistor_SMD:R_0402_1005Metric, F.Cu at (122.5, 130.6)
- added R10: 27R, Resistor_SMD:R_0402_1005Metric, F.Cu at (113.8, 130.1)
- added R10: 27R, Resistor_SMD:R_0402_1005Metric, F.Cu at (141.8, 130.1)
- added R10: 27R, Resistor_SMD:R_0402_1005Metric, F.Cu at (156.2, 81.0)
- added R11: 200R, Resistor_SMD:R_0603_1608Metric, F.Cu at (128.6, 129.8)
- added R11: 200R, Resistor_SMD:R_0603_1608Metric, F.Cu at (156.6, 129.8)
- added R11: 200R, Resistor_SMD:R_0603_1608Metric, F.Cu at (141.4, 81.2)
- added R12: 1R, Resistor_SMD:R_0402_1005Metric, F.Cu at (159.1, 129.7)
- added R12: 1R, Resistor_SMD:R_0402_1005Metric, F.Cu at (131.1, 129.7)
- added R12: 1R, Resistor_SMD:R_0402_1005Metric, F.Cu at (138.9, 81.3)
- added R15: 200K, Resistor_SMD:R_0402_1005Metric, F.Cu at (151.6, 118.5)
- added R15: 200K, Resistor_SMD:R_0402_1005Metric, F.Cu at (146.4, 92.5)
- added R15: 200K, Resistor_SMD:R_0402_1005Metric, F.Cu at (123.6, 118.5)
- added R16: 100K, Resistor_SMD:R_0402_1005Metric, F.Cu at (147.5, 119.3)
- added R16: 100K, Resistor_SMD:R_0402_1005Metric, F.Cu at (119.5, 119.3)
- added R16: 100K, Resistor_SMD:R_0402_1005Metric, F.Cu at (150.5, 91.7)
- added R17: 470R, Resistor_SMD:R_0402_1005Metric, F.Cu at (157.2, 78.2)
- added R17: 470R, Resistor_SMD:R_0402_1005Metric, F.Cu at (112.8, 132.8)
- added R17: 470R, Resistor_SMD:R_0402_1005Metric, F.Cu at (140.8, 132.8)
- added R2: 1K, Resistor_SMD:R_0402_1005Metric, F.Cu at (154.0, 114.2)
- added R2: 1K, Resistor_SMD:R_0402_1005Metric, F.Cu at (126.0, 114.2)
- added R2: 1K, Resistor_SMD:R_0402_1005Metric, F.Cu at (144.0, 96.8)
- added R4: 470R, Resistor_SMD:R_0402_1005Metric, F.Cu at (109.5, 109.0)
- added R4: 470R, Resistor_SMD:R_0402_1005Metric, F.Cu at (137.5, 109.0)
- added R4: 470R, Resistor_SMD:R_0402_1005Metric, F.Cu at (160.5, 102.0)
- added R9: 27R, Resistor_SMD:R_0402_1005Metric, F.Cu at (154.7, 81.0)
- added R9: 27R, Resistor_SMD:R_0402_1005Metric, F.Cu at (115.3, 130.1)
- added R9: 27R, Resistor_SMD:R_0402_1005Metric, F.Cu at (143.3, 130.1)
- added REF**: DrillHole_0.6mm, MountingHole:DrillHole_0.6mm, F.Cu at (136.2, 130.3)
- added REF**: DrillHole_0.6mm, MountingHole:DrillHole_0.6mm, F.Cu at (156.3, 75.2)
- added REF**: DrillHole_0.6mm, MountingHole:DrillHole_0.6mm, F.Cu at (164.2, 130.7)
- added REF**: DrillHole_0.6mm, MountingHole:DrillHole_0.6mm, F.Cu at (136.2, 98.0)
- added REF**: Fiducial, TestPoint:Fiducial, F.Cu at (103.0, 71.3)
- added REF**: DrillHole_0.6mm, MountingHole:DrillHole_0.6mm, F.Cu at (161.8, 100.7)
- added REF**: DrillHole_0.6mm, MountingHole:DrillHole_0.6mm, F.Cu at (159.0, 75.2)
- added REF**: DrillHole_0.6mm, MountingHole:DrillHole_0.6mm, F.Cu at (128.3, 135.8)
- added REF**: DrillHole_0.6mm, MountingHole:DrillHole_0.6mm, F.Cu at (133.8, 100.7)
- added REF**: DrillHole_0.6mm, MountingHole:DrillHole_0.6mm, F.Cu at (156.3, 72.8)
- added REF**: DrillHole_0.6mm, MountingHole:DrillHole_0.6mm, F.Cu at (164.2, 129.8)
- added REF**: DrillHole_0.6mm, MountingHole:DrillHole_0.6mm, F.Cu at (105.8, 98.9)
- added REF**: DrillHole_0.6mm, MountingHole:DrillHole_0.6mm, F.Cu at (136.8, 104.8)
- added REF**: DrillHole_0.6mm, MountingHole:DrillHole_0.6mm, F.Cu at (105.8, 130.7)
- added REF**: DrillHole_0.6mm, MountingHole:DrillHole_0.6mm, F.Cu at (133.8, 98.9)
- added REF**: DrillHole_0.6mm, MountingHole:DrillHole_0.6mm, F.Cu at (136.2, 112.1)
- added REF**: DrillHole_0.6mm, MountingHole:DrillHole_0.6mm, F.Cu at (139.9, 138.2)
- added REF**: DrillHole_0.6mm, MountingHole:DrillHole_0.6mm, F.Cu at (164.2, 98.0)
- added REF**: DrillHole_0.6mm, MountingHole:DrillHole_0.6mm, F.Cu at (108.2, 110.9)
- added REF**: DrillHole_0.6mm, MountingHole:DrillHole_0.6mm, F.Cu at (111.9, 135.8)
- added REF**: DrillHole_0.6mm, MountingHole:DrillHole_0.6mm, F.Cu at (164.2, 99.8)
- added REF**: DrillHole_0.6mm, MountingHole:DrillHole_0.6mm, F.Cu at (157.2, 75.2)
- added REF**: DrillHole_0.6mm, MountingHole:DrillHole_0.6mm, F.Cu at (111.0, 75.2)
- added REF**: DrillHole_0.6mm, MountingHole:DrillHole_0.6mm, F.Cu at (136.2, 129.4)
- added REF**: DrillHole_0.6mm, MountingHole:DrillHole_0.6mm, F.Cu at (161.8, 99.8)
- added REF**: DrillHole_0.6mm, MountingHole:DrillHole_0.6mm, F.Cu at (157.2, 135.8)
- added REF**: DrillHole_0.6mm, MountingHole:DrillHole_0.6mm, F.Cu at (140.8, 72.8)
- added REF**: DrillHole_0.6mm, MountingHole:DrillHole_0.6mm, F.Cu at (131.0, 138.2)
- added REF**: DrillHole_0.6mm, MountingHole:DrillHole_0.6mm, F.Cu at (161.8, 110.0)
- added REF**: DrillHole_0.6mm, MountingHole:DrillHole_0.6mm, F.Cu at (108.2, 82.7)
- added REF**: DrillHole_0.6mm, MountingHole:DrillHole_0.6mm, F.Cu at (133.2, 104.8)
- added REF**: DrillHole_0.6mm, MountingHole:DrillHole_0.6mm, F.Cu at (133.8, 129.4)
- added REF**: DrillHole_0.6mm, MountingHole:DrillHole_0.6mm, F.Cu at (111.9, 75.2)
- added REF**: DrillHole_0.6mm, MountingHole:DrillHole_0.6mm, F.Cu at (159.0, 138.2)
- added REF**: DrillHole_0.6mm, MountingHole:DrillHole_0.6mm, F.Cu at (112.8, 75.2)
- added REF**: DrillHole_0.6mm, MountingHole:DrillHole_0.6mm, F.Cu at (140.8, 138.2)
- added REF**: DrillHole_0.6mm, MountingHole:DrillHole_0.6mm, F.Cu at (108.2, 130.7)
- added REF**: DrillHole_0.6mm, MountingHole:DrillHole_0.6mm, F.Cu at (128.3, 138.2)
- added REF**: DrillHole_0.6mm, MountingHole:DrillHole_0.6mm, F.Cu at (164.2, 100.7)
- added REF**: DrillHole_0.6mm, MountingHole:DrillHole_0.6mm, F.Cu at (133.8, 80.4)
- added REF**: DrillHole_0.6mm, MountingHole:DrillHole_0.6mm, F.Cu at (133.8, 104.2)
- added REF**: DrillHole_0.6mm, MountingHole:DrillHole_0.6mm, F.Cu at (164.2, 80.0)
- added REF**: DrillHole_0.6mm, MountingHole:DrillHole_0.6mm, F.Cu at (156.3, 135.8)
- added REF**: DrillHole_0.6mm, MountingHole:DrillHole_0.6mm, F.Cu at (108.2, 81.8)
- added REF**: DrillHole_0.6mm, MountingHole:DrillHole_0.6mm, F.Cu at (141.7, 75.2)
- added REF**: DrillHole_0.6mm, MountingHole:DrillHole_0.6mm, F.Cu at (161.8, 81.8)
- added REF**: DrillHole_0.6mm, MountingHole:DrillHole_0.6mm, F.Cu at (164.2, 128.9)
- added REF**: DrillHole_0.6mm, MountingHole:DrillHole_0.6mm, F.Cu at (164.2, 110.9)
- added REF**: DrillHole_0.6mm, MountingHole:DrillHole_0.6mm, F.Cu at (136.2, 80.4)
- added REF**: DrillHole_0.6mm, MountingHole:DrillHole_0.6mm, F.Cu at (161.8, 98.9)
- added REF**: DrillHole_0.6mm, MountingHole:DrillHole_0.6mm, F.Cu at (111.0, 135.8)
- added REF**: DrillHole_0.6mm, MountingHole:DrillHole_0.6mm, F.Cu at (108.2, 128.9)
- added REF**: DrillHole_0.6mm, MountingHole:DrillHole_0.6mm, F.Cu at (108.2, 112.7)
- added REF**: DrillHole_0.6mm, MountingHole:DrillHole_0.6mm, F.Cu at (136.2, 79.5)
- added REF**: DrillHole_0.6mm, MountingHole:DrillHole_0.6mm, F.Cu at (133.8, 98.0)
- added REF**: DrillHole_0.6mm, MountingHole:DrillHole_0.6mm, F.Cu at (105.8, 80.0)
- added REF**: Fiducial, TestPoint:Fiducial, F.Cu at (167.0, 71.3)
- added REF**: DrillHole_0.6mm, MountingHole:DrillHole_0.6mm, F.Cu at (139.9, 72.8)
- added REF**: DrillHole_0.6mm, MountingHole:DrillHole_0.6mm, F.Cu at (131.0, 135.8)
- added REF**: DrillHole_0.6mm, MountingHole:DrillHole_0.6mm, F.Cu at (130.1, 138.2)
- added REF**: DrillHole_0.6mm, MountingHole:DrillHole_0.6mm, F.Cu at (112.8, 138.2)
- added REF**: DrillHole_0.6mm, MountingHole:DrillHole_0.6mm, F.Cu at (133.8, 110.3)
- added REF**: DrillHole_0.6mm, MountingHole:DrillHole_0.6mm, F.Cu at (136.2, 111.2)
- added REF**: DrillHole_0.6mm, MountingHole:DrillHole_0.6mm, F.Cu at (130.1, 72.8)
- added REF**: DrillHole_0.6mm, MountingHole:DrillHole_0.6mm, F.Cu at (136.2, 81.3)
- added REF**: DrillHole_0.6mm, MountingHole:DrillHole_0.6mm, F.Cu at (157.2, 138.2)
- added REF**: DrillHole_0.6mm, MountingHole:DrillHole_0.6mm, F.Cu at (140.8, 135.8)
- added REF**: DrillHole_0.6mm, MountingHole:DrillHole_0.6mm, F.Cu at (141.7, 135.8)
- added REF**: DrillHole_0.6mm, MountingHole:DrillHole_0.6mm, F.Cu at (161.8, 128.9)
- added REF**: DrillHole_0.6mm, MountingHole:DrillHole_0.6mm, F.Cu at (108.2, 80.9)
- added REF**: DrillHole_0.6mm, MountingHole:DrillHole_0.6mm, F.Cu at (156.3, 138.2)
- added REF**: DrillHole_0.6mm, MountingHole:DrillHole_0.6mm, F.Cu at (136.2, 99.8)
- added REF**: DrillHole_0.6mm, MountingHole:DrillHole_0.6mm, F.Cu at (161.8, 128.0)
- added REF**: DrillHole_0.6mm, MountingHole:DrillHole_0.6mm, F.Cu at (111.9, 138.2)
- added REF**: DrillHole_0.6mm, MountingHole:DrillHole_0.6mm, F.Cu at (158.1, 72.8)
- added REF**: DrillHole_0.6mm, MountingHole:DrillHole_0.6mm, F.Cu at (108.2, 110.0)
- added REF**: DrillHole_0.6mm, MountingHole:DrillHole_0.6mm, F.Cu at (159.0, 72.8)
- added REF**: DrillHole_0.6mm, MountingHole:DrillHole_0.6mm, F.Cu at (161.8, 80.0)
- added REF**: DrillHole_0.6mm, MountingHole:DrillHole_0.6mm, F.Cu at (157.2, 72.8)
- added REF**: DrillHole_0.6mm, MountingHole:DrillHole_0.6mm, F.Cu at (133.8, 112.1)
- added REF**: DrillHole_0.6mm, MountingHole:DrillHole_0.6mm, F.Cu at (161.8, 98.0)
- added REF**: DrillHole_0.6mm, MountingHole:DrillHole_0.6mm, F.Cu at (161.8, 112.7)
- added REF**: DrillHole_0.6mm, MountingHole:DrillHole_0.6mm, F.Cu at (105.8, 128.9)
- added REF**: Fiducial, TestPoint:Fiducial, F.Cu at (103.0, 139.2)
- added REF**: DrillHole_0.6mm, MountingHole:DrillHole_0.6mm, F.Cu at (111.9, 72.8)
- added REF**: DrillHole_0.6mm, MountingHole:DrillHole_0.6mm, F.Cu at (113.7, 75.2)
- added REF**: DrillHole_0.6mm, MountingHole:DrillHole_0.6mm, F.Cu at (141.7, 72.8)
- added REF**: DrillHole_0.6mm, MountingHole:DrillHole_0.6mm, F.Cu at (108.2, 99.8)
- added REF**: DrillHole_0.6mm, MountingHole:DrillHole_0.6mm, F.Cu at (164.2, 98.9)
- added REF**: Fiducial, TestPoint:Fiducial, F.Cu at (135.0, 71.3)
- added REF**: DrillHole_0.6mm, MountingHole:DrillHole_0.6mm, F.Cu at (105.8, 128.0)
- added REF**: Fiducial, TestPoint:Fiducial, F.Cu at (135.0, 139.2)
- added REF**: DrillHole_0.6mm, MountingHole:DrillHole_0.6mm, F.Cu at (164.2, 112.7)
- added REF**: DrillHole_0.6mm, MountingHole:DrillHole_0.6mm, F.Cu at (133.8, 111.2)
- added REF**: DrillHole_0.6mm, MountingHole:DrillHole_0.6mm, F.Cu at (129.2, 75.2)
- added REF**: DrillHole_0.6mm, MountingHole:DrillHole_0.6mm, F.Cu at (131.0, 75.2)
- added REF**: DrillHole_0.6mm, MountingHole:DrillHole_0.6mm, F.Cu at (108.2, 100.7)
- added REF**: Fiducial, TestPoint:Fiducial, F.Cu at (167.0, 139.2)
- added REF**: DrillHole_0.6mm, MountingHole:DrillHole_0.6mm, F.Cu at (158.1, 75.2)
- added REF**: DrillHole_0.6mm, MountingHole:DrillHole_0.6mm, F.Cu at (131.0, 72.8)
- added REF**: DrillHole_0.6mm, MountingHole:DrillHole_0.6mm, F.Cu at (111.0, 138.2)
- added REF**: DrillHole_0.6mm, MountingHole:DrillHole_0.6mm, F.Cu at (161.8, 111.8)
- added REF**: DrillHole_0.6mm, MountingHole:DrillHole_0.6mm, F.Cu at (105.8, 112.7)
- added REF**: DrillHole_0.6mm, MountingHole:DrillHole_0.6mm, F.Cu at (141.7, 138.2)
- added REF**: DrillHole_0.6mm, MountingHole:DrillHole_0.6mm, F.Cu at (105.8, 81.8)
- added REF**: DrillHole_0.6mm, MountingHole:DrillHole_0.6mm, F.Cu at (164.2, 81.8)
- added REF**: DrillHole_0.6mm, MountingHole:DrillHole_0.6mm, F.Cu at (136.2, 113.0)
- added REF**: DrillHole_0.6mm, MountingHole:DrillHole_0.6mm, F.Cu at (130.1, 75.2)
- added REF**: DrillHole_0.6mm, MountingHole:DrillHole_0.6mm, F.Cu at (105.8, 110.9)
- added REF**: DrillHole_0.6mm, MountingHole:DrillHole_0.6mm, F.Cu at (133.8, 79.5)
- added REF**: DrillHole_0.6mm, MountingHole:DrillHole_0.6mm, F.Cu at (112.8, 72.8)
- added REF**: DrillHole_0.6mm, MountingHole:DrillHole_0.6mm, F.Cu at (136.2, 98.9)
- added REF**: DrillHole_0.6mm, MountingHole:DrillHole_0.6mm, F.Cu at (158.1, 135.8)
- added REF**: DrillHole_0.6mm, MountingHole:DrillHole_0.6mm, F.Cu at (161.8, 110.9)
- added REF**: DrillHole_0.6mm, MountingHole:DrillHole_0.6mm, F.Cu at (129.2, 72.8)
- added REF**: DrillHole_0.6mm, MountingHole:DrillHole_0.6mm, F.Cu at (136.8, 106.2)
- added REF**: DrillHole_0.6mm, MountingHole:DrillHole_0.6mm, F.Cu at (164.2, 111.8)
- added REF**: DrillHole_0.6mm, MountingHole:DrillHole_0.6mm, F.Cu at (112.8, 135.8)
- added REF**: DrillHole_0.6mm, MountingHole:DrillHole_0.6mm, F.Cu at (133.8, 131.2)
- added REF**: DrillHole_0.6mm, MountingHole:DrillHole_0.6mm, F.Cu at (139.0, 138.2)
- added REF**: DrillHole_0.6mm, MountingHole:DrillHole_0.6mm, F.Cu at (113.7, 72.8)
- added REF**: DrillHole_0.6mm, MountingHole:DrillHole_0.6mm, F.Cu at (136.2, 82.2)
- added REF**: DrillHole_0.6mm, MountingHole:DrillHole_0.6mm, F.Cu at (133.8, 106.8)
- added REF**: DrillHole_0.6mm, MountingHole:DrillHole_0.6mm, F.Cu at (130.1, 135.8)
- added REF**: DrillHole_0.6mm, MountingHole:DrillHole_0.6mm, F.Cu at (129.2, 135.8)
- added REF**: DrillHole_0.6mm, MountingHole:DrillHole_0.6mm, F.Cu at (164.2, 80.9)
- added REF**: DrillHole_0.6mm, MountingHole:DrillHole_0.6mm, F.Cu at (133.8, 113.0)
- added REF**: DrillHole_0.6mm, MountingHole:DrillHole_0.6mm, F.Cu at (133.8, 128.5)
- added REF**: DrillHole_0.6mm, MountingHole:DrillHole_0.6mm, F.Cu at (113.7, 135.8)
- added REF**: DrillHole_0.6mm, MountingHole:DrillHole_0.6mm, F.Cu at (108.2, 98.9)
- added REF**: DrillHole_0.6mm, MountingHole:DrillHole_0.6mm, F.Cu at (136.2, 106.8)
- added REF**: DrillHole_0.6mm, MountingHole:DrillHole_0.6mm, F.Cu at (161.8, 129.8)
- added REF**: DrillHole_0.6mm, MountingHole:DrillHole_0.6mm, F.Cu at (105.8, 100.7)
- added REF**: DrillHole_0.6mm, MountingHole:DrillHole_0.6mm, F.Cu at (136.2, 128.5)
- added REF**: DrillHole_0.6mm, MountingHole:DrillHole_0.6mm, F.Cu at (133.8, 130.3)
- added REF**: DrillHole_0.6mm, MountingHole:DrillHole_0.6mm, F.Cu at (133.8, 82.2)
- added REF**: DrillHole_0.6mm, MountingHole:DrillHole_0.6mm, F.Cu at (158.1, 138.2)
- added REF**: DrillHole_0.6mm, MountingHole:DrillHole_0.6mm, F.Cu at (108.2, 80.0)
- added REF**: DrillHole_0.6mm, MountingHole:DrillHole_0.6mm, F.Cu at (161.8, 130.7)
- added REF**: DrillHole_0.6mm, MountingHole:DrillHole_0.6mm, F.Cu at (139.0, 72.8)
- added REF**: DrillHole_0.6mm, MountingHole:DrillHole_0.6mm, F.Cu at (111.0, 72.8)
- added REF**: DrillHole_0.6mm, MountingHole:DrillHole_0.6mm, F.Cu at (133.2, 106.2)
- added REF**: DrillHole_0.6mm, MountingHole:DrillHole_0.6mm, F.Cu at (105.8, 82.7)
- added REF**: DrillHole_0.6mm, MountingHole:DrillHole_0.6mm, F.Cu at (136.2, 100.7)
- added REF**: DrillHole_0.6mm, MountingHole:DrillHole_0.6mm, F.Cu at (139.9, 75.2)
- added REF**: DrillHole_0.6mm, MountingHole:DrillHole_0.6mm, F.Cu at (139.0, 135.8)
- added REF**: DrillHole_0.6mm, MountingHole:DrillHole_0.6mm, F.Cu at (140.8, 75.2)
- added REF**: DrillHole_0.6mm, MountingHole:DrillHole_0.6mm, F.Cu at (108.2, 111.8)
- added REF**: DrillHole_0.6mm, MountingHole:DrillHole_0.6mm, F.Cu at (136.2, 131.2)
- added REF**: DrillHole_0.6mm, MountingHole:DrillHole_0.6mm, F.Cu at (113.7, 138.2)
- added REF**: DrillHole_0.6mm, MountingHole:DrillHole_0.6mm, F.Cu at (108.2, 129.8)
- added REF**: DrillHole_0.6mm, MountingHole:DrillHole_0.6mm, F.Cu at (108.2, 128.0)
- added REF**: DrillHole_0.6mm, MountingHole:DrillHole_0.6mm, F.Cu at (105.8, 98.0)
- added REF**: DrillHole_0.6mm, MountingHole:DrillHole_0.6mm, F.Cu at (108.2, 98.0)
- added REF**: DrillHole_0.6mm, MountingHole:DrillHole_0.6mm, F.Cu at (105.8, 129.8)
- added REF**: DrillHole_0.6mm, MountingHole:DrillHole_0.6mm, F.Cu at (105.8, 80.9)
- added REF**: DrillHole_0.6mm, MountingHole:DrillHole_0.6mm, F.Cu at (136.2, 110.3)
- added REF**: DrillHole_0.6mm, MountingHole:DrillHole_0.6mm, F.Cu at (129.2, 138.2)
- added REF**: DrillHole_0.6mm, MountingHole:DrillHole_0.6mm, F.Cu at (161.8, 80.9)
- added REF**: DrillHole_0.6mm, MountingHole:DrillHole_0.6mm, F.Cu at (164.2, 110.0)
- added REF**: DrillHole_0.6mm, MountingHole:DrillHole_0.6mm, F.Cu at (105.8, 111.8)
- added REF**: DrillHole_0.6mm, MountingHole:DrillHole_0.6mm, F.Cu at (128.3, 72.8)
- added REF**: DrillHole_0.6mm, MountingHole:DrillHole_0.6mm, F.Cu at (128.3, 75.2)
- added REF**: DrillHole_0.6mm, MountingHole:DrillHole_0.6mm, F.Cu at (136.2, 104.2)
- added REF**: DrillHole_0.6mm, MountingHole:DrillHole_0.6mm, F.Cu at (139.9, 135.8)
- added REF**: DrillHole_0.6mm, MountingHole:DrillHole_0.6mm, F.Cu at (139.0, 75.2)
- added REF**: DrillHole_0.6mm, MountingHole:DrillHole_0.6mm, F.Cu at (105.8, 110.0)
- added REF**: DrillHole_0.6mm, MountingHole:DrillHole_0.6mm, F.Cu at (164.2, 128.0)
- added REF**: DrillHole_0.6mm, MountingHole:DrillHole_0.6mm, F.Cu at (133.8, 99.8)
- added REF**: DrillHole_0.6mm, MountingHole:DrillHole_0.6mm, F.Cu at (133.8, 81.3)
- added REF**: DrillHole_0.6mm, MountingHole:DrillHole_0.6mm, F.Cu at (159.0, 135.8)
- added REF**: DrillHole_0.6mm, MountingHole:DrillHole_0.6mm, F.Cu at (105.8, 99.8)
- added REF**: DrillHole_0.6mm, MountingHole:DrillHole_0.6mm, F.Cu at (161.8, 82.7)
- added REF**: DrillHole_0.6mm, MountingHole:DrillHole_0.6mm, F.Cu at (164.2, 82.7)
- added S1: K3-1203S-E1, JLCPCB:SW-SMD_K3-1203S-E1, F.Cu at (140.6, 102.0)
- added S1: K3-1203S-E1, JLCPCB:SW-SMD_K3-1203S-E1, F.Cu at (129.4, 109.0)
- added S1: K3-1203S-E1, JLCPCB:SW-SMD_K3-1203S-E1, F.Cu at (157.4, 109.0)
- added TP1: TestPoint, TestPoint:TestPoint_Pad_1.5x1.5mm, F.Cu at (143.3, 76.0)
- added TP1: TestPoint, TestPoint:TestPoint_Pad_1.5x1.5mm, F.Cu at (154.7, 135.0)
- added TP1: TestPoint, TestPoint:TestPoint_Pad_1.5x1.5mm, F.Cu at (126.7, 135.0)
- added TP2: TestPoint, TestPoint:TestPoint_Pad_1.5x1.5mm, B.Cu at (143.3, 76.0)
- added TP2: TestPoint, TestPoint:TestPoint_Pad_1.5x1.5mm, B.Cu at (126.7, 135.0)
- added TP2: TestPoint, TestPoint:TestPoint_Pad_1.5x1.5mm, B.Cu at (154.7, 135.0)
- added TP3: TestPoint, TestPoint:TestPoint_Pad_1.5x1.5mm, F.Cu at (115.3, 135.0)
- added TP3: TestPoint, TestPoint:TestPoint_Pad_1.5x1.5mm, F.Cu at (143.3, 135.0)
- added TP3: TestPoint, TestPoint:TestPoint_Pad_1.5x1.5mm, F.Cu at (154.7, 76.0)
- added TP4: TestPoint, TestPoint:TestPoint_Pad_1.5x1.5mm, B.Cu at (143.3, 135.0)
- added TP4: TestPoint, TestPoint:TestPoint_Pad_1.5x1.5mm, B.Cu at (154.7, 76.0)
- added TP4: TestPoint, TestPoint:TestPoint_Pad_1.5x1.5mm, B.Cu at (115.3, 135.0)
- added TP5: BOOT, TestPoint:TestPoint_Pad_1.0x1.0mm, B.Cu at (127.7, 113.7)
- added TP5: BOOT, TestPoint:TestPoint_Pad_1.0x1.0mm, B.Cu at (142.3, 97.3)
- added TP5: BOOT, TestPoint:TestPoint_Pad_1.0x1.0mm, B.Cu at (155.7, 113.7)
- added TP7: RST2, TestPoint:TestPoint_Pad_1.0x1.0mm, B.Cu at (147.9, 83.5)
- added TP7: RST2, TestPoint:TestPoint_Pad_1.0x1.0mm, B.Cu at (150.1, 127.5)
- added TP7: RST2, TestPoint:TestPoint_Pad_1.0x1.0mm, B.Cu at (122.1, 127.5)
- added TP8: RST1, TestPoint:TestPoint_Pad_1.0x1.0mm, B.Cu at (140.9, 121.3)
- added TP8: RST1, TestPoint:TestPoint_Pad_1.0x1.0mm, B.Cu at (157.1, 89.7)
- added TP8: RST1, TestPoint:TestPoint_Pad_1.0x1.0mm, B.Cu at (112.9, 121.3)
- added U1: AP7366EA-3.3, Package_DFN_QFN:Diodes_UDFN2020-6_Type-F, F.Cu at (140.1, 78.5)
- added U1: AP7366EA-3.3, Package_DFN_QFN:Diodes_UDFN2020-6_Type-F, F.Cu at (157.9, 132.5)
- added U1: AP7366EA-3.3, Package_DFN_QFN:Diodes_UDFN2020-6_Type-F, F.Cu at (129.9, 132.5)
- added U2: RP2040, Package_DFN_QFN:QFN-56-1EP_7x7mm_P0.4mm_EP3.2x3.2mm, F.Cu at (154.0, 124.3)
- added U2: RP2040, Package_DFN_QFN:QFN-56-1EP_7x7mm_P0.4mm_EP3.2x3.2mm, F.Cu at (144.0, 86.7)
- added U2: RP2040, Package_DFN_QFN:QFN-56-1EP_7x7mm_P0.4mm_EP3.2x3.2mm, F.Cu at (126.0, 124.3)
- added U3: W25Q16JVUXIQ, SnapEDA:IC_W25Q16JVUXIQ_TR, F.Cu at (159.9, 122.2)
- added U3: W25Q16JVUXIQ, SnapEDA:IC_W25Q16JVUXIQ_TR, F.Cu at (131.9, 122.2)
- added U3: W25Q16JVUXIQ, SnapEDA:IC_W25Q16JVUXIQ_TR, F.Cu at (138.1, 88.8)
- added U4: RP2040, Package_DFN_QFN:QFN-56-1EP_7x7mm_P0.4mm_EP3.2x3.2mm, F.Cu at (116.0, 124.3)
- added U4: RP2040, Package_DFN_QFN:QFN-56-1EP_7x7mm_P0.4mm_EP3.2x3.2mm, F.Cu at (144.0, 124.3)
- added U4: RP2040, Package_DFN_QFN:QFN-56-1EP_7x7mm_P0.4mm_EP3.2x3.2mm, F.Cu at (154.0, 86.7)
- added U5: W25Q16JVUXIQ, SnapEDA:IC_W25Q16JVUXIQ_TR, F.Cu at (150.5, 80.8)
- added U5: W25Q16JVUXIQ, SnapEDA:IC_W25Q16JVUXIQ_TR, F.Cu at (147.5, 130.2)
- added U5: W25Q16JVUXIQ, SnapEDA:IC_W25Q16JVUXIQ_TR, F.Cu at (119.5, 130.2)
- added X1: SX2M12.000M20F30TNN, Oscillator:Oscillator_SMD_ECS_2520MV-xxx-xx-4Pin_2.5x2.0mm, F.Cu at (138.0, 120.8)
- added X1: SX2M12.000M20F30TNN, Oscillator:Oscillator_SMD_ECS_2520MV-xxx-xx-4Pin_2.5x2.0mm, F.Cu at (160.0, 90.2)
- added X1: SX2M12.000M20F30TNN, Oscillator:Oscillator_SMD_ECS_2520MV-xxx-xx-4Pin_2.5x2.0mm, F.Cu at (110.0, 120.8)
- Q2: footprint Package_DFN_QFN:Diodes_DFN1006-3 -> Package_TO_SOT_SMD:SOT-723
- R10, R9: footprint Resistor_SMD:R_0201_0603Metric -> Resistor_SMD:R_0402_1005Metric
- S1: value Würth_450404015514 -> K3-1203S-E1; footprint SnapEDA:450404015514 -> JLCPCB:SW-SMD_K3-1203S-E1
- X1: value ECS-2520MVLC-120-CM-TR -> SX2M12.000M20F30TNN
- moved S1 22.3 mm to (112.5, 102.0), turned to 0 degrees
- moved C13 21.8 mm to (125.3, 80.8)
- moved R9 21.8 mm to (126.7, 81.0)
- moved C21 21.8 mm to (131.0, 87.3)
- moved C19 21.8 mm to (121.0, 87.8)
- moved D1 21.8 mm to (132.0, 104.2)
- moved R2 21.8 mm to (116.0, 96.8)
- moved U1 21.8 mm to (112.1, 78.5)
- moved U3 21.8 mm to (110.1, 88.8)
- moved C10 21.8 mm to (112.5, 91.7)
- moved C12 21.8 mm to (128.0, 92.0)
- moved C16 21.8 mm to (121.0, 83.8)
- moved C2 21.8 mm to (111.6, 76.2)
- moved C5 21.8 mm to (121.0, 86.2)
- moved C6 21.8 mm to (111.0, 85.8)
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Connections:
- Q3 pad 1: SWCLK -> GPIO2
- Q3 pad 2: GPIO2 -> DEV_ENABLE
- Q3 pad 6: DEV_ENABLE -> SWCLK
Routing:
- net +3V3: track 64.4 -> 237.1 mm, vias 16 -> 64
- net VBUS: track 40.8 -> 154.0 mm, vias 2 -> 8
- net LED_EN: track 28.2 -> 110.9 mm, vias 2 -> 8
- net SWCLK: track 22.9 -> 90.0 mm, vias 3 -> 12
- net /Development Board Section/RUN: track 19.4 -> 86.3 mm, vias 2 -> 8
- net SWDIO: track 23.3 -> 88.6 mm, vias 2 -> 8
- net OSC_OUT: track 19.7 -> 78.4 mm
- net /Development Board Section/1V1_CORE: track 18.9 -> 76.2 mm
- net /Debug Probe Section/1V1_CORE: track 16.1 -> 67.6 mm
- net GPIO_ADC0: track 18.1 -> 68.6 mm, vias 2 -> 8
- net GPIO3: track 13.8 -> 63.7 mm, vias 1 -> 4
- net GPIO5: track 16.0 -> 65.4 mm, vias 1 -> 4
- net GPIO_ADC1: track 16.9 -> 65.3 mm, vias 2 -> 8
- net GPIO4: track 14.1 -> 55.9 mm, vias 1 -> 4
- net /Development Board Section/GPIO_ADC3: track 11.8 -> 51.0 mm, vias 2 -> 8
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Other:
- board size 26 x 30 mm -> 70 x 75 mm
