File: Electrical/KiCad_templates/Expansion_Card_Retrofit/Expansion_Card_Retrofit.kicad_sch (KiCad schematic)
At the start: 15 parts, among them J1 Conn 10P, P1 USB_C_Plug_USB2.0, Q3 Q_Dual_NPN_NPN_C2E2C1E1B1B2, U1 AP7366EA-3.3, X1 ECS-2520MVLC-120-CM-TR

Commit message: Production design v1 finished
Parts:
- Q3: symbol Device:Q_Dual_NPN_NPN_C2E2C1E1B1B2 -> Device:Q_Dual_NPN_NPN_E1B1C2E2B2C1
- S1: value Würth_450404015514 -> K3-1203S-E1; footprint SnapEDA:450404015514 -> JLCPCB:SW-SMD_K3-1203S-E1
- X1: value ECS-2520MVLC-120-CM-TR -> SX2M12.000M20F30TNN
Connections:
- net DEV_ENABLE: now also Q3.2 (B1), Q3.5 (B2); no longer Q3.5 (B1), Q3.6 (B2)
- net GPIO2: now also Q3.1 (E1); no longer Q3.2 (E2)
- net GPIO3: now also Q3.4 (E2); no longer Q3.4 (E1)
- net SWCLK: now also Q3.6 (C1); no longer Q3.1 (C2)
- net SWDIO: now also Q3.3 (C2); no longer Q3.3 (C1)
Other:
- moved on the sheet: Q3A, Q3B, X1
Changed lines of the file:
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@@
   )
   (no_connect (at 57.15 45.72))
-  (no_connect (at 31.115 118.745))
+  (no_connect (at 33.02 115.57))
   (no_connect (at 222.885 101.6))
   (wire (pts (xy 241.935 154.94) (xy 247.015 154.94))
@@
     (stroke (width 0) (type default))
   )
-  (wire (pts (xy 41.275 108.585) (xy 41.275 111.125))
+  (wire (pts (xy 43.18 105.41) (xy 43.18 107.95))
     (stroke (width 0) (type default))
   )
@@
     (stroke (width 0) (type default))
   )
-  (wire (pts (xy 41.275 126.365) (xy 41.275 128.905))
+  (wire (pts (xy 43.18 123.19) (xy 43.18 125.73))
     (stroke (width 0) (type default))
   )
@@
     (stroke (width 0) (type default))
   )
-  (text "Oscillator" (at 33.02 99.06 0)
+  (text "Oscillator" (at 34.29 97.79 0)
     (effects (font (size 2.54 2.54)) (justify left bottom))
   )
@@
     )
   )
-  (global_label "OSC_OUT" (shape output) (at 51.435 118.745 0) (fields_autoplaced)
+  (global_label "OSC_OUT" (shape output) (at 53.34 115.57 0) (fields_autoplaced)
     (effects (font (size 1.27 1.27)) (justify left))
-    (property "Intersheetrefs" "${INTERSHEET_REFS}" (at 62.1722 118.745 0)
+    (property "Intersheetrefs" "${INTERSHEET_REFS}" (at 64.0772 115.57 0)
       (effects (font (size 1.27 1.27)) (justify left) hide)
     )
@@
     )
   )
-  (symbol (lib_id "power:+3V3") (at 41.275 108.585 0) (unit 1)
+  (symbol (lib_id "power:+3V3") (at 43.18 105.41 0) (unit 1)
     (in_bom yes) (on_board yes) (dnp no) (fields_autoplaced)
-    (property "Reference" "#PWR046" (at 41.275 112.395 0)
-      (effects (font (size 1.27 1.27)) hide)
-    )
-    (property "Value" "+3V3" (at 41.275 104.14 0)
-      (effects (font (size 1.27 1.27)))
-    )
-    (property "Footprint" "" (at 41.275 108.585 0)
-      (effects (font (size 1.27 1.27)) hide)
-    )
-    (property "Datasheet" "" (at 41.275 108.585 0)
+    (property "Reference" "#PWR046" (at 43.18 109.22 0)
+      (effects (font (size 1.27 1.27)) hide)
+    )
+    (property "Value" "+3V3" (at 43.18 100.965 0)
+      (effects (font (size 1.27 1.27)))
+    )
+    (property "Footprint" "" (at 43.18 105.41 0)
+      (effects (font (size 1.27 1.27)) hide)
+    )
+    (property "Datasheet" "" (at 43.18 105.41 0)
       (effects (font (size 1.27 1.27)) hide)
     )
@@
     )
   )
-  (symbol (lib_id "Oscillator:ECS-2520MV-xxx-xx") (at 41.275 118.745 0) (unit 1)
-    (in_bom yes) (on_board yes) (dnp no)
-    (property "Reference" "X1" (at 44.45 108.585 0)
-      (effects (font (size 1.27 1.27)) (justify left))
-    )
-    (property "Value" "ECS-2520MVLC-120-CM-TR" (at 44.45 111.125 0)
-      (effects (font (size 1.27 1.27)) (justify left))
-    )
-    (property "Footprint" "Oscillator:Oscillator_SMD_ECS_2520MV-xxx-xx-4Pin_2.5x2.0mm" (at 52.705 127.635 0)
-      (effects (font (size 1.27 1.27)) hide)
-    )
-    (property "Datasheet" "https://www.ecsxtal.com/store/pdf/ECS-2520MV.pdf" (at 36.83 115.57 0)
+  (symbol (lib_id "Oscillator:ECS-2520MV-xxx-xx") (at 43.18 115.57 0) (unit 1)
+    (in_bom yes) (on_board yes) (dnp no)
+    (property "Reference" "X1" (at 46.355 105.41 0)
+      (effects (font (size 1.27 1.27)) (justify left))
+    )
+    (property "Value" "SX2M12.000M20F30TNN" (at 46.355 107.95 0)
+      (effects (font (size 1.27 1.27)) (justify left))
+    )
+    (property "Footprint" "Oscillator:Oscillator_SMD_ECS_2520MV-xxx-xx-4Pin_2.5x2.0mm" (at 54.61 124.46 0)
+      (effects (font (size 1.27 1.27)) hide)
+    )
+    (property "Datasheet" "https://www.ecsxtal.com/store/pdf/ECS-2520MV.pdf" (at 38.735 112.395 0)
       (effects (font (size 1.27 1.27)) hide)
     )
@@
       (effects (font (size 1.27 1.27)) (justify right))
     )
-    (property "Value" "Würth_450404015514" (at 223.52 92.71 0)
+    (property "Value" "K3-1203S-E1" (at 223.52 92.71 0)
       (effects (font (size 1.27 1.27)) (justify right))
     )
-    (property "Footprint" "SnapEDA:450404015514" (at 227.965 99.06 0)
+    (property "Footprint" "JLCPCB:SW-SMD_K3-1203S-E1" (at 227.965 99.06 0)
       (effects (font (size 1.27 1.27)) (justify bottom) hide)
     )
@@
     )
   )
-  (symbol (lib_id "Device:Q_Dual_NPN_NPN_C2E2C1E1B1B2") (at 243.205 106.68 90) (mirror x) (unit 2)
-    (in_bom yes) (on_board yes) (dnp no)
-    (property "Reference" "Q3" (at 238.76 113.03 90)
+  (symbol (lib_id "Device:Q_Dual_NPN_NPN_E1B1C2E2B2C1") (at 243.205 125.73 90) (mirror x) (unit 2)
+    (in_bom yes) (on_board yes) (dnp no)
+    (property "Reference" "Q3" (at 238.76 132.08 90)
       (effects (font (size 1.27 1.27)) (justify right))
     )
-    (property "Value" "Q_Dual_NPN_NPN_C2E2C1E1B1B2" (at 238.76 115.57 90)
+    (property "Value" "Q_Dual_NPN_NPN_C2E2C1E1B1B2" (at 238.76 134.62 90)
       (effects (font (size 1.27 1.27)) (justify right))
     )
-    (property "Footprint" "digikey-footprints:SOT-363" (at 240.665 111.76 0)
-      (effects (font (size 1.27 1.27)) hide)
-    )
-    (property "Datasheet" "~" (at 243.205 106.68 0)
-      (effects (font (size 1.27 1.27)) hide)
-    )
+    (property "Footprint" "digikey-footprints:SOT-363" (at 240.665 130.81 0)
+      (effects (font (size 1.27 1.27)) hide)
+    )
+    (property "Datasheet" "~" (at 243.205 125.73 0)
+      (effects (font (size 1.27 1.27)) hide)
+    )
+    (pin "1")
+    (pin "2")
+    (pin "6")
     (pin "3")
     (pin "4")
     (pin "5")
+    (instances
+      (project "Expansion_Card_Retrofit"
+        (path "/fd9cf59f-f670-406e-98d4-36112036cae5"
+          (reference "Q3") (unit 2)
+        )
+      )
+    )
+  )
+  (symbol (lib_id "Device:Q_Dual_NPN_NPN_E1B1C2E2B2C1") (at 243.205 106.68 90) (mirror x) (unit 1)
+    (in_bom yes) (on_board yes) (dnp no)
+    (property "Reference" "Q3" (at 238.76 113.03 90)
+      (effects (font (size 1.27 1.27)) (justify right))
+    )
+    (property "Value" "Q_Dual_NPN_NPN_C2E2C1E1B1B2" (at 238.76 115.57 90)
+      (effects (font (size 1.27 1.27)) (justify right))
+    )
+    (property "Footprint" "digikey-footprints:SOT-363" (at 240.665 111.76 0)
+      (effects (font (size 1.27 1.27)) hide)
+    )
+    (property "Datasheet" "~" (at 243.205 106.68 0)
+      (effects (font (size 1.27 1.27)) hide)
+    )
     (pin "1")
     (pin "2")
     (pin "6")
-    (instances
-      (project "Expansion_Card_Retrofit"
-        (path "/fd9cf59f-f670-406e-98d4-36112036cae5"
-          (reference "Q3") (unit 2)
-        )
-      )
-    )
-  )
-  (symbol (lib_id "Device:Q_Dual_NPN_NPN_C2E2C1E1B1B2") (at 243.205 125.73 90) (mirror x) (unit 1)
-    (in_bom yes) (on_board yes) (dnp no)
-    (property "Reference" "Q3" (at 238.76 132.08 90)
-      (effects (font (size 1.27 1.27)) (justify right))
-    )
-    (property "Value" "Q_Dual_NPN_NPN_C2E2C1E1B1B2" (at 238.76 134.62 90)
-      (effects (font (size 1.27 1.27)) (justify right))
-    )
-    (property "Footprint" "digikey-footprints:SOT-363" (at 240.665 130.81 0)
-      (effects (font (size 1.27 1.27)) hide)
-    )
-    (property "Datasheet" "~" (at 243.205 125.73 0)
-      (effects (font (size 1.27 1.27)) hide)
-    )
     (pin "3")
     (pin "4")
     (pin "5")
-    (pin "1")
-    (pin "2")
-    (pin "6")
     (instances
       (project "Expansion_Card_Retrofit"
@@
     )
   )
-  (symbol (lib_id "power:GND") (at 41.275 128.905 0) (unit 1)
+  (symbol (lib_id "power:GND") (at 43.18 125.73 0) (unit 1)
     (in_bom yes) (on_board yes) (dnp no) (fields_autoplaced)
-    (property "Reference" "#PWR047" (at 41.275 135.255 0)
-      (effects (font (size 1.27 1.27)) hide)
-    )
-    (property "Value" "GND" (at 41.275 133.35 0)
-      (effects (font (size 1.27 1.27)))
-    )
-    (property "Footprint" "" (at 41.275 128.905 0)
-      (effects (font (size 1.27 1.27)) hide)
-    )
-    (property "Datasheet" "" (at 41.275 128.905 0)
+    (property "Reference" "#PWR047" (at 43.18 132.08 0)
+      (effects (font (size 1.27 1.27)) hide)
+    )
+    (property "Value" "GND" (at 43.18 130.175 0)
+      (effects (font (size 1.27 1.27)))
+    )
+    (property "Footprint" "" (at 43.18 125.73 0)
+      (effects (font (size 1.27 1.27)) hide)
+    )
+    (property "Datasheet" "" (at 43.18 125.73 0)
       (effects (font (size 1.27 1.27)) hide)
     )
@@
     )
   )
-  (sheet (at 111.125 148.59) (size 36.195 34.925) (fields_autoplaced)
+  (sheet (at 111.125 144.78) (size 36.195 34.925) (fields_autoplaced)
     (stroke (width 0.1524) (type solid))
     (fill (color 0 0 0 0.0000))
-    (property "Sheetname" "Debug Probe Section" (at 111.125 147.8784 0)
+    (property "Sheetname" "Debug Probe Section" (at 111.125 144.0684 0)
       (effects (font (size 1.27 1.27)) (justify left bottom))
     )
-    (property "Sheetfile" "debug_probe_section.kicad_sch" (at 111.125 184.0996 0)
+    (property "Sheetfile" "debug_probe_section.kicad_sch" (at 111.125 180.2896 0)
       (effects (font (size 1.27 1.27)) (justify left top))
     )
@@
     )
   )
-  (sheet (at 37.465 149.225) (size 38.735 36.195) (fields_autoplaced)
+  (sheet (at 37.465 145.415) (size 38.735 36.195) (fields_autoplaced)
     (stroke (width 0.1524) (type solid))
     (fill (color 0 0 0 0.0000))
-    (property "Sheetname" "Development Board Section" (at 37.465 148.5134 0)
+    (property "Sheetname" "Development Board Section" (at 37.465 144.7034 0)
       (effects (font (size 1.27 1.27)) (justify left bottom))
     )
-    (property "Sheetfile" "dev_board_section.kicad_sch" (at 37.465 186.0046 0)
+    (property "Sheetfile" "dev_board_section.kicad_sch" (at 37.465 182.1946 0)
       (effects (font (size 1.27 1.27)) (justify left top))
     )
