File: Electrical/KiCad_templates/Expansion_Card_Retrofit/debug_probe_section.kicad_sch (KiCad schematic)
At the start: 18 parts, among them U3 W25Q16JVUXIQ, U4 RP2040

Commit message: Production design v1 finished
Parts:
- R10, R9: footprint Resistor_SMD:R_0201_0603Metric -> Resistor_SMD:R_0402_1005Metric
- TP5: value TestPoint -> BOOT
- TP8: value TestPoint -> RST1
Changed lines of the file:
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@@
       (effects (font (size 1.27 1.27)))
     )
-    (property "Value" "TestPoint" (at 131.318 54.61 90)
+    (property "Value" "BOOT" (at 131.318 54.61 90)
       (effects (font (size 1.27 1.27)))
     )
@@
       (effects (font (size 1.27 1.27)) (justify left))
     )
-    (property "Value" "TestPoint" (at 52.07 69.85 0)
+    (property "Value" "RST1" (at 52.07 69.85 0)
       (effects (font (size 1.27 1.27)) (justify left))
     )
@@
       (effects (font (size 1.27 1.27)))
     )
-    (property "Footprint" "Resistor_SMD:R_0201_0603Metric" (at 49.53 78.613 90)
+    (property "Footprint" "Resistor_SMD:R_0402_1005Metric" (at 49.53 78.613 90)
       (effects (font (size 1.27 1.27)) hide)
     )
@@
       (effects (font (size 1.27 1.27)))
     )
-    (property "Footprint" "Resistor_SMD:R_0201_0603Metric" (at 49.53 86.233 90)
-      (effects (font (size 1.27 1.27)) hide)
-    )
+    (property "Footprint" "Resistor_SMD:R_0402_1005Metric" (at 49.53 86.233 90)
+      (effects (font (size 1.27 1.27)) hide)
+    )
